Commit message: Diseño del Robot con URDF completado

File: robot/pandt_robot.urdf (robot description, URDF)
Before this commit: robot pandt_robot, 1 links, 0 joints
Links:
- added link camera; visual box size=0.2 0.2 0.2
- added link der_body; visual box size=0.3 0.05 0.6
- added link izq_body; visual box size=0.3 0.05 0.6
- added link pan_body; visual box size=0.3 0.3 0.8
- added link tilt_body; visual box size=0.3 0.3 0.3
- added link world
- link base_link: geometry visual cylinder length=0.05 radius=0.5
Joints:
- added joint CameraBody: type fixed, parent tilt_body, child camera, origin xyz=0 0 0 rpy=0 0 0, axis 0 1 0
- added joint DerBody: type fixed, parent tilt_body, child der_body, origin xyz=0 0 0 rpy=0 0 0, axis 0 1 0
- added joint IzqBody: type fixed, parent tilt_body, child izq_body, origin xyz=0 0 0 rpy=0 0 0, axis 0 1 0
- added joint Pan: type continuous, parent base_link, child pan_body, origin xyz=0 0 0.40 rpy=0 0 0, axis 0 0 1
- added joint Tilt: type continuous, parent pan_body, child tilt_body, origin xyz=0 0 0.3 rpy=0 0 0, axis 0 1 0
- added joint fixed: type fixed, parent world, child base_link

Commit message: Cambiando el tilt para que tenga límites

File: robot/pandt_robot.urdf (robot description, URDF)
Before this commit: robot pandt_robot, 7 links, 6 joints
Joints:
- joint Tilt: limit (none) -> lower=-2 upper=2 effort=10 velocity=1.0; type continuous -> revolute
